File: muon.kicad_pcb (KiCad board)
At the start: 2 copper layers, 33.5 x 10 mm, 9 parts, among them J1 HRO_TYPE-C-31-M-12, J2 SM04B-SRSS-TB, U1 TPD4E05U06DQA

Commit message: Update to A2 revision
Parts:
- MH1, MH2: value Pad-M3 -> Pad-M2.5; footprint locallib:MountingHole-M3-Simple -> locallib:MountingHole-M2.5-Simple
- moved MH1 0.50 mm to (81.5, 55.0)
- moved MH2 0.50 mm to (55.0, 55.0)
- moved J2 0.10 mm to (61.5, 56.9)
- moved U1 0.10 mm to (66.8, 57.1)
Other:
- board size 33.5 x 10 mm -> 31.5 x 10 mm
- board text added: "USB PCB A2"
- board text removed: "USB PCB A1"
