File: muon.kicad_sch (KiCad schematic)
At the start: 9 parts, among them J1 HRO_TYPE-C-31-M-12, J2 SM04B-SRSS-TB, U1 TPD4E05U06DQA

Commit message: Update to A2 revision
Parts:
- MH1, MH2: value Pad-M3 -> Pad-M2.5; footprint locallib:MountingHole-M3-Simple -> locallib:MountingHole-M2.5-Simple
Changed lines of the file:
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@@
 			)
 		)
-		(property "Value" "Pad-M3"
+		(property "Value" "Pad-M2.5"
 			(at 185.42 77.4699 0)
 			(effects
@@
 			)
 		)
-		(property "Footprint" "locallib:MountingHole-M3-Simple"
+		(property "Footprint" "locallib:MountingHole-M2.5-Simple"
 			(at 182.88 76.2 0)
 			(effects
@@
 			)
 		)
-		(property "Value" "Pad-M3"
+		(property "Value" "Pad-M2.5"
 			(at 185.42 85.0899 0)
 			(effects
@@
 			)
 		)
-		(property "Footprint" "locallib:MountingHole-M3-Simple"
+		(property "Footprint" "locallib:MountingHole-M2.5-Simple"
 			(at 182.88 83.82 0)
 			(effects
