File: Var-A/muon.kicad_pcb (KiCad board)
At the start: 2 copper layers, 31.5 x 10 mm, 9 parts, among them J1 HRO_TYPE-C-31-M-12, J2 SM04B-SRSS-TB, U1 TPD4E05U06DQA

Commit message: Make B variant
Other:
- board text added: "A2"
- board text removed: "USB PCB A2"
